File: tpf-fedefarfan/arduino-nano-a.kicad_pcb (KiCad board)
At the start: 2 copper layers, 23 x 48.8 mm, 34 parts, among them J1 USB_B_Mini, J2 Conn_02x03_Counter_Clockwise, J3 Conn_01x15, J4 Conn_01x15, SW1 SW_Push, U1 LM1117-5.0, U2 FT232RL, U3 ATmega328P-A, Y1 Crystal

Commit message: Trabajo Final
Parts:
- moved FID2 0.31 mm to (105.7, 105.2)
- moved J1 0.19 mm to (111.8, 105.0)
Routing:
- net GND: track 139.9 -> 139.2 mm
Changed lines of the file:
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@@
     (property "Sheetname" "")
     (attr smd)
-    (fp_text reference "SW1" (at 0 -2.25) (layer "F.SilkS")
+    (fp_text reference "SW1" (at -2.0574 -2.8956) (layer "F.SilkS")
       (effects (font (size 1 1) (thickness 0.15)))
     )
@@
     (property "Sheetname" "")
     (attr smd)
-    (fp_text reference "R4" (at 0 -1.65 -90) (layer "F.SilkS")
+    (fp_text reference "R4" (at 0.3048 1.3716 -90) (layer "F.SilkS")
       (effects (font (size 1 1) (thickness 0.15)))
     )
@@
     (property "Sheetname" "")
     (attr exclude_from_pos_files)
-    (fp_text reference "H3" (at 0 -2.75) (layer "F.SilkS")
+    (fp_text reference "H3" (at 1.7272 1.8542) (layer "F.SilkS")
       (effects (font (size 1 1) (thickness 0.15)))
     )
@@
     (property "Sheetname" "")
     (attr smd)
-    (fp_text reference "R6" (at 0 -1.65 90) (layer "F.SilkS")
+    (fp_text reference "R6" (at 0.0254 -1.524 90) (layer "F.SilkS")
       (effects (font (size 1 1) (thickness 0.15)))
     )
@@
     (property "Sheetname" "")
     (attr exclude_from_pos_files)
-    (fp_text reference "H4" (at 0 -2.75) (layer "F.SilkS")
+    (fp_text reference "H4" (at -1.524 1.8796) (layer "F.SilkS")
       (effects (font (size 1 1) (thickness 0.15)))
     )
@@
     (property "Sheetname" "")
     (attr exclude_from_pos_files)
-    (fp_text reference "H2" (at 0 -2.75) (layer "F.SilkS")
+    (fp_text reference "H2" (at -3.2512 -1.0922) (layer "F.SilkS")
       (effects (font (size 1 1) (thickness 0.15)))
     )
@@
     (property "Sheetname" "")
     (attr smd)
-    (fp_text reference "R3" (at 0 -1.65 -90) (layer "F.SilkS")
+    (fp_text reference "R3" (at 0 1.524 -90) (layer "F.SilkS")
       (effects (font (size 1 1) (thickness 0.15)))
     )
@@
     (property "Sheetname" "")
     (attr smd)
-    (fp_text reference "R5" (at 0 -1.65 -90) (layer "F.SilkS")
+    (fp_text reference "R5" (at 1.4986 1.3208 -90) (layer "F.SilkS")
       (effects (font (size 1 1) (thickness 0.15)))
     )
@@
     (property "Sheetname" "")
     (attr smd)
-    (fp_text reference "R7" (at 0 -1.65 90) (layer "F.SilkS")
+    (fp_text reference "R7" (at 2.9558 0.735 90) (layer "F.SilkS")
       (effects (font (size 1 1) (thickness 0.15)))
     )
@@
     (property "Sheetname" "")
     (attr smd)
-    (fp_text reference "C8" (at 0 -1.68 -90) (layer "F.SilkS")
+    (fp_text reference "C8" (at -2.921 1.3462 -90) (layer "F.SilkS")
       (effects (font (size 1 1) (thickness 0.15)))
     )
@@
     (property "Sheetname" "")
     (attr smd)
-    (fp_text reference "D2" (at 0 -1.65 90) (layer "F.SilkS")
+    (fp_text reference "D2" (at -0.499 -1.8542 90) (layer "F.SilkS")
       (effects (font (size 1 1) (thickness 0.15)))
     )
@@
     (property "Sheetname" "")
     (attr smd)
-    (fp_text reference "FID1" (at 0 -2) (layer "F.SilkS")
+    (fp_text reference "FID1" (at 0 2.3114) (layer "F.SilkS")
       (effects (font (size 1 1) (thickness 0.15)))
     )
@@
     (property "Sheetname" "")
     (attr through_hole)
-    (fp_text reference "J2" (at 1.27 -2.33 90) (layer "F.SilkS")
+    (fp_text reference "J2" (at 2.667 7.62 90) (layer "F.SilkS")
       (effects (font (size 1 1) (thickness 0.15)))
     )
@@
     (property "Sheetname" "")
     (attr exclude_from_pos_files)
-    (fp_text reference "H1" (at 0 -2.75) (layer "F.SilkS")
+    (fp_text reference "H1" (at 2.8702 -1.1938) (layer "F.SilkS")
       (effects (font (size 1 1) (thickness 0.15)))
     )
@@
     (property "Sheetname" "")
     (attr smd)
-    (fp_text reference "D5" (at 0 -1.65 90) (layer "F.SilkS")
+    (fp_text reference "D5" (at 2.1336 -1.651 90) (layer "F.SilkS")
       (effects (font (size 1 1) (thickness 0.15)))
     )
@@
   )
   (footprint "Fiducial:Fiducial_1mm_Mask2mm" (layer "F.Cu")
-    (at 105.7148 104.8512)
+    (at 105.664 105.156)
     (descr "Circular Fiducial, 1mm bare copper, 2mm soldermask opening (Level A)")
     (tags "fiducial")
@@
     (property "Sheetname" "")
     (attr smd)
-    (fp_text reference "FID2" (at 0 -2) (layer "F.SilkS")
+    (fp_text reference "FID2" (at -0.3048 -4.5212) (layer "F.SilkS")
       (effects (font (size 1 1) (thickness 0.15)))
     )
@@
   )
   (footprint "Connector_USB:USB_Mini-B_Lumberg_2486_01_Horizontal" (layer "F.Cu")
-    (at 111.76 104.775)
+    (at 111.76 104.97)
     (descr "USB Mini-B 5-pin SMD connector, http://downloads.lumberg.com/datenblaetter/en/2486_01.pdf")
     (tags "USB USB_B USB_Mini connector")
@@
     (property "Sheetname" "")
     (attr smd)
-    (fp_text reference "C3" (at 0 1.85) (layer "B.SilkS")
+    (fp_text reference "C3" (at -0.4064 -2.0066) (layer "B.SilkS")
       (effects (font (size 1 1) (thickness 0.15)) (justify mirror))
     )
@@
     (property "Sheetname" "")
     (attr smd)
-    (fp_text reference "C6" (at 0 1.75 90) (layer "B.SilkS")
+    (fp_text reference "C6" (at -3.6576 0 90) (layer "B.SilkS")
       (effects (font (size 1 1) (thickness 0.15)) (justify mirror))
     )
@@
     (property "Sheetname" "")
     (attr smd)
-    (fp_text reference "C4" (at 0 1.85) (layer "B.SilkS")
+    (fp_text reference "C4" (at -2.3114 2.0214) (layer "B.SilkS")
       (effects (font (size 1 1) (thickness 0.15)) (justify mirror))
     )
@@
     (property "Sheetname" "")
     (attr through_hole)
-    (fp_text reference "J3" (at 0 2.33) (layer "B.SilkS")
+    (fp_text reference "J3" (at -4.318 3.7592) (layer "B.SilkS")
       (effects (font (size 1 1) (thickness 0.15)) (justify mirror))
     )
@@
     (property "Sheetname" "")
     (attr smd)
-    (fp_text reference "C5" (at 0 1.68 270) (layer "B.SilkS")
+    (fp_text reference "C5" (at 2.7393 1.68 270) (layer "B.SilkS")
       (effects (font (size 1 1) (thickness 0.15)) (justify mirror))
     )
@@
     (property "Sheetname" "")
     (attr through_hole)
-    (fp_text reference "J4" (at 0 2.33) (layer "B.SilkS")
+    (fp_text reference "J4" (at 3.9624 3.7134) (layer "B.SilkS")
       (effects (font (size 1 1) (thickness 0.15)) (justify mirror))
     )
@@
     (property "Sheetname" "")
     (attr smd)
-    (fp_text reference "R1" (at 0 1.65 270) (layer "B.SilkS")
+    (fp_text reference "R1" (at 2.8194 1.6526 270) (layer "B.SilkS")
       (effects (font (size 1 1) (thickness 0.15)) (justify mirror))
     )
@@
       (effects (font (size 1 1) (thickness 0.15)) (justify mirror))
     )
-    (fp_text value "FT232RL" (at 0 -6.25) (layer "B.Fab")
+    (fp_text value "FT232RL" (at 0 -7.62) (layer "B.Fab")
       (effects (font (size 1 1) (thickness 0.15)) (justify mirror))
     )
@@
   (segment (start 112.3657 82.474818) (end 112.3657 81.153) (width 0.25) (layer "B.Cu") (net 2))
   (segment (start 109.6374 101.335) (end 110.479 101.335) (width 0.25) (layer "B.Cu") (net 2))
-  (segment (start 114.7441 81.8388) (end 114.2361 81.3308) (width 0.25) (layer "B.Cu") (net 2))
   (segment (start 116.7384 98.9884) (end 116.7384 101.7167) (width 0.25) (layer "B.Cu") (net 2))
   (segment (start 110.0582 88.6714) (end 110.0582 93.4212) (width 0.25) (layer "B.Cu") (net 2))
@@
   (segment (start 104.2532 102.0942) (end 104.2532 102.256594) (width 0.25) (layer "B.Cu") (net 16))
   (segment (start 104.2532 102.256594) (end 105.062103 103.065497) (width 0.25) (layer "B.Cu") (net 16))
-  (segment (start 105.283 68.4276) (end 105.172095 68.4276) (width 0.25) (layer "B.Cu") (net 16))
   (segment (start 104.2532 102.0942) (end 104.2532 69.4574) (width 0.25) (layer "B.Cu") (net 16))
   (segment (start 114.3 68.453) (end 115.874502 68.453) (width 0.25) (layer "F.Cu") (net 17))
