File: tpf-fedefarfan/arduino-nano-a.kicad_sch (KiCad schematic)
At the start: 29 parts, among them J1 USB_B_Mini, J2 Conn_02x03_Counter_Clockwise, J3 Conn_01x15, J4 Conn_01x15, SW1 SW_Push, U1 LM1117-5.0, U2 FT232RL, U3 ATmega328P-A, Y1 Crystal

Commit message: Trabajo Final
Parts:
- added FID1, FID2: Fiducial, Fiducial:Fiducial_1mm_Mask2mm, symbol Mechanical:Fiducial
- added H1, H2, H3, H4: MountingHole, MountingHole:MountingHole_2.2mm_M2_ISO7380, symbol Mechanical:MountingHole
Connections:
- net GND: now also SW1.2; no longer SW1.1
- net RESET: now also R7.2, SW1.1, U3.29 (~{RESET}/PC6)
- net CBUS0: now reaches R3.2, U2.23 (CBUS0)
- net CBUS1: now reaches R4.2, U2.22 (CBUS1)
Other:
- note added: "SEÑALES"
- note removed: "AUTO SELECTOR 5V"
- title: ARDUINO NANO -> REPLICA ARDUINO NANO
- moved on the sheet: C1, C2, C3, C4, C5, C6, C7, C8, D1, D2, D3, D4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

Commit message: Trabajo Final
Connections:
- net +3.3V renamed +3V3
Changed lines of the file:
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@@
     (pin "2")
   )
-  (symbol (lib_name "FT232RL_1") (lib_id "Interface_USB:FT232RL") (at 73.66 139.7 0) (unit 1)
+  (symbol (lib_id "Interface_USB:FT232RL") (at 73.66 139.7 0) (unit 1)
     (in_bom yes) (on_board yes) (fields_autoplaced)
     (property "Reference" "U2" (id 0) (at 78.2194 113.03 0)
